File: hardware/main_board/mini_robot.sch (EAGLE design)
At the start: 77 parts, among them IC2 MCP601OT, IC3 MCP73811/2, Q1 BSS123, Q2 12MHz, U1 ISL29125, U2 DRV8836DSSR, U3 ATMEGA328-AU

Commit message: pcb
Connections:
- net +3V3: no longer ISP1.VCC
- net VCC: now also ISP1.VCC
